File: hardware/firmware-programmer/onboard-signal-router/onboard-signal-router.sch (KiCad schematic (older format))
At the start: 36 parts

Commit message: mostly completed routing and board layout.
Parts:
- removed U? (x8): 74LS125, symbol 74xx:74LS125
- added C1, C10, C11, C2, C3, C4, C5, C6, C7, C8, C9: 0.1uF, Capacitor_SMD:C_0603_1608Metric_Pad1.05x0.95mm_HandSolder, symbol Device:C_Small
- added unit 5 of U1
- added unit 6 of U1
- added unit 1 of U5
- added unit 2 of U5
- added unit 3 of U5
- added unit 4 of U5
- added unit 4 of U6
- added unit 3 of U6
- added unit 2 of U6
- added unit 1 of U6
- added unit 1 of U7
- added unit 2 of U7
- added unit 3 of U7
- added unit 4 of U7
- added unit 7 of U7
- added U8: MAX14851AEE+, MAX14851-PLUS:MAX14851AEE&plus_, symbol MAX14851-PLUS:MAX14851AEE+
- added U9: MAX14930DAWE+, MAX14930DAWE_PLUS:MAX14930DAWE&plus_, symbol MAX14930DAWE_PLUS:MAX14930DAWE+
- J1: renamed from J?; footprint (none) -> Connector_Dsub:DSUB-9_Male_Vertical_P2.77x2.84mm_MountingHoles
- J2: renamed from J?; value Conn_02x05_Top_Bottom -> RCS-ISP; footprint (none) -> Connector_IDC:IDC-Header_2x05_P2.54mm_Vertical; symbol Connector_Generic:Conn_02x05_Top_Bottom -> Connector_Generic:Conn_02x05_Odd_Even
- J3: renamed from J?; value Conn_02x05_Top_Bottom -> TCS-ISP; footprint (none) -> Connector_IDC:IDC-Header_2x05_P2.54mm_Vertical; symbol Connector_Generic:Conn_02x05_Top_Bottom -> Connector_Generic:Conn_02x05_Odd_Even
- J4: renamed from J?; value Conn_02x05_Top_Bottom -> DCS-ISP; footprint (none) -> Connector_IDC:IDC-Header_2x05_P2.54mm_Vertical; symbol Connector_Generic:Conn_02x05_Top_Bottom -> Connector_Generic:Conn_02x05_Odd_Even
- U1, U2, U3, U4, U5, U6, U7: renamed from U?; footprint (none) -> Package_SO:SOIC-14_3.9x8.7mm_P1.27mm
Connections:
- net BC1_ISO: now reaches U1.1
- net BC1_ISO: now also U2.2, U2.9, U1.13, U9.14 (OUTB1)
- net ~BC1_ISO: now reaches U1.2
- net ~BC1_ISO: now also U2.5
- net BC0_ISO: now reaches U1.3
- net BC0_ISO: now also U2.6, U2.8, U1.11, U9.13 (OUTB2)
- net ~BC0_ISO: now reaches U1.4
- net ~BC0_ISO: now also U2.1
- net GNDD: now reaches U1.5
- net GNDD: now also J2.10 (Pin_10), J2.4 (Pin_4), J2.6 (Pin_6), J2.8 (Pin_8), J3.10 (Pin_10), J3.4 (Pin_4), J3.6 (Pin_6), J3.8 (Pin_8), J4.10 (Pin_10), J4.4 (Pin_4), J4.6 (Pin_6), J4.8 (Pin_8), U1.6, U1.7 (VSS), U1.8, U1.9, U2.12, U2.13, U2.7 (VSS), U3.7 (VSS), U4.7 (GND), U5.7 (GND), U6.7 (GND), C1.1, C10.1, C11.1, C2.1, C3.1, C4.1, C5.1, C6.1, C9.1, U7.7 (VSS), U8.10 (I/OB2), U8.12 (INB2), U8.9 (GNDB), U9.11 (OUTB4), U9.12 (OUTB3), U9.15 (GNDB), U9.9 (GNDB)
- net at U7.10: now also U3.2
- net at U7.11: now also U3.11, U7.13, U7.1
- net at U7.12: now also U3.6
- net +5VD: now reaches U1.14 (VDD)
- net +5VD: now also J2.2 (Pin_2), J3.2 (Pin_2), J4.2 (Pin_2), U2.14 (VDD), U3.14 (VDD), U4.14 (VCC), U5.14 (VCC), U6.14 (VCC), C1.2, C10.2, C11.2, C2.2, C3.2, C4.2, C5.2, C6.2, C9.2, U7.14 (VDD), U8.16 (VCCB), U9.10 (ENB), U9.16 (VDDB)
- net at U2.3: now also U3.5
- net at U2.4: now also U3.1
- net at U2.10: now also U3.8
- net at U3.12: now also U1.10
- net at U3.13: now also U1.12
- net DCS_BSEL: now reaches U3.10
- net DCS_BSEL: now also U7.9
- net at U3.9: now also U7.2
- net TCS_BSEL: now reaches U3.4
- net TCS_BSEL: now also U7.5
- net RCS_BSEL: now reaches U3.3
- net RCS_BSEL: now also U7.3
- net GNDPWR: now reaches J1.0 (PAD)
- net GNDPWR: now also J1.7, J1.9, C7.2, C8.2, U8.5 (OUTA2), U8.7 (I/OA2), U8.8 (GNDA), U9.2 (GNDA), U9.5 (INA3), U9.6 (INA4), U9.8 (GNDA)
- net VBUS: now reaches J1.1
- net VBUS: now also C7.1, C8.1, U8.1 (VCCA), U9.1 (VDDA)
- net MOSI: now reaches J1.2
- net MOSI: now also U8.2 (INA1)
- net SCK: now reaches J1.3
- net SCK: now also U8.3 (INA2)
- net MISO: now reaches J1.4
- net MISO: now also U8.6 (I/OA1)
- net BC0: now reaches J1.5
- net BC0: now also U9.4 (INA2)
- net BC1: now reaches J1.6
- net BC1: now also U9.3 (INA1)
- net ~RST: now reaches J1.8
- net ~RST: now also U8.4 (OUTA1)
- net RCS_MOSI: now reaches J2.1 (Pin_1)
- net RCS_MOSI: now also U4.3
- net ~RCS_RST: now reaches J2.5 (Pin_5)
- net ~RCS_RST: now also U4.8
- net RCS_SCK: now reaches J2.7 (Pin_7)
- net RCS_SCK: now also U4.6
- net RCS_MISO: now reaches J2.9 (Pin_9)
- net RCS_MISO: now also U4.12
- net TCS_MOSI: now reaches J3.1 (Pin_1)
- net TCS_MOSI: now also U5.3
- net ~TCS_RST: now reaches J3.5 (Pin_5)
- net ~TCS_RST: now also U5.11
- net TCS_SCK: now reaches J3.7 (Pin_7)
- net TCS_SCK: now also U5.6
- net TCS_MISO: now reaches J3.9 (Pin_9)
- net TCS_MISO: now also U5.9
- net DCS_MOSI: now reaches J4.1 (Pin_1)
- net DCS_MOSI: now also U6.3
- net ~DCS_RST: now reaches J4.5 (Pin_5)
- net ~DCS_RST: now also U6.8
- net DCS_SCK: now reaches J4.7 (Pin_7)
- net DCS_SCK: now also U6.6
- net DCS_MISO: now reaches J4.9 (Pin_9)
- net DCS_MISO: now also U6.12
- net ~RCS_BSEL: now reaches U4.1
- net ~RCS_BSEL: now also U4.10, U4.13, U4.4, U7.4
- net MOSI_ISO: now reaches U4.2
- net MOSI_ISO: now also U5.2, U6.2, U8.15 (OUTB1)
- net SCK_ISO: now reaches U4.5
- net SCK_ISO: now also U5.5, U6.5, U8.14 (OUTB2)
- net ~RST_ISO: now reaches U4.9
- net ~RST_ISO: now also U5.12, U6.9, U8.11 (I/OB1)
- net MISO_ISO: now reaches U4.11
- net MISO_ISO: now also U5.8, U6.11, U8.13 (INB1)
- new net ~DCS_BSEL: U6.1, U6.10, U6.13, U6.4, U7.8
- new net ~TCS_BSEL: U5.1, U5.10, U5.13, U5.4, U7.6
- no-connect marks 0 -> 5
Other:
- moved on the sheet: J2, J3, J4, U1A, U1B, U1C, U1D, U1G, U2A, U2B, U2C, U2D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
